File: boards/raspberry_pi/TempHumiditySensorRaspberryPi.sch (EAGLE design)
At the start: 10 parts, among them J1 GPIO4, J2 GPIO17, J3 GPIO22, J4 GPIO23, J5 GPIO24, J6 GPIO25, J7 GPIO8, J8 GPIO7

Commit message: MacroFab files and BOM
Added BOMs for use with eagle-config and production files for MacroFab.

DSB
Parts:
- J1, J2, J3, J4, J5, J6, J7, J8: PARTNO (none) -> 5555164-1
- SV1: PARTNO (none) -> SBH11-PBPC-D13-ST-BK
Changed lines of the file:
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@@
 <?xml version="1.0" encoding="utf-8"?>
 <!DOCTYPE eagle SYSTEM "eagle.dtd">
-<eagle version="6.6.0">
+<eagle version="8.5.0">
 <drawing>
 <settings>
 <setting alwaysvectorfont="no"/>
+<setting keepoldvectorfont="yes"/>
 <setting verticaltext="up"/>
 </settings>
-<grid distance="0.1" unitdist="inch" unit="inch" style="lines" multiple="1" display="no" altdistance="0.01" altunitdist="inch" altunit="inch"/>
+<grid distance="0.05" unitdist="inch" unit="inch" style="lines" multiple="1" display="no" altdistance="0.01" altunitdist="inch" altunit="inch"/>
 <layers>
 <layer number="1" name="Top" color="4" fill="1" visible="no" active="no"/>
@@
 </classes>
 <parts>
-<part name="SV1" library="con-harting-ml" deviceset="ML26" device="" value="RPi"/>
-<part name="J1" library="con-amp" deviceset="555164-1" device="" value="GPIO4"/>
-<part name="J2" library="con-amp" deviceset="555164-1" device="" value="GPIO17"/>
-<part name="J3" library="con-amp" deviceset="555164-1" device="" value="GPIO22"/>
-<part name="J4" library="con-amp" deviceset="555164-1" device="" value="GPIO23"/>
-<part name="J5" library="con-amp" deviceset="555164-1" device="" value="GPIO24"/>
-<part name="J8" library="con-amp" deviceset="555164-1" device="" value="GPIO7"/>
-<part name="J7" library="con-amp" deviceset="555164-1" device="" value="GPIO8"/>
-<part name="J6" library="con-amp" deviceset="555164-1" device="" value="GPIO25"/>
+<part name="SV1" library="con-harting-ml" deviceset="ML26" device="" value="RPi">
+<attribute name="PARTNO" value="SBH11-PBPC-D13-ST-BK"/>
+</part>
+<part name="J1" library="con-amp" deviceset="555164-1" device="" value="GPIO4">
+<attribute name="PARTNO" value="5555164-1"/>
+</part>
+<part name="J2" library="con-amp" deviceset="555164-1" device="" value="GPIO17">
+<attribute name="PARTNO" value="5555164-1"/>
+</part>
+<part name="J3" library="con-amp" deviceset="555164-1" device="" value="GPIO22">
+<attribute name="PARTNO" value="5555164-1"/>
+</part>
+<part name="J4" library="con-amp" deviceset="555164-1" device="" value="GPIO23">
+<attribute name="PARTNO" value="5555164-1"/>
+</part>
+<part name="J5" library="con-amp" deviceset="555164-1" device="" value="GPIO24">
+<attribute name="PARTNO" value="5555164-1"/>
+</part>
+<part name="J8" library="con-amp" deviceset="555164-1" device="" value="GPIO7">
+<attribute name="PARTNO" value="5555164-1"/>
+</part>
+<part name="J7" library="con-amp" deviceset="555164-1" device="" value="GPIO8">
+<attribute name="PARTNO" value="5555164-1"/>
+</part>
+<part name="J6" library="con-amp" deviceset="555164-1" device="" value="GPIO25">
+<attribute name="PARTNO" value="5555164-1"/>
+</part>
 <part name="+3V1" library="supply1" deviceset="+3V3" device=""/>
 <part name="GND1" library="supply1" deviceset="GND" device=""/>
@@
 </plain>
 <instances>
-<instance part="SV1" gate="1" x="66.04" y="68.58" rot="MR180"/>
-<instance part="J1" gate="G$1" x="12.7" y="116.84" rot="R180"/>
-<instance part="J2" gate="G$1" x="12.7" y="83.82" rot="R180"/>
-<instance part="J3" gate="G$1" x="12.7" y="50.8" rot="R180"/>
-<instance part="J4" gate="G$1" x="12.7" y="12.7" rot="R180"/>
-<instance part="J5" gate="G$1" x="-27.94" y="5.08" rot="R180"/>
-<instance part="J8" gate="G$1" x="-25.4" y="50.8" rot="R180"/>
-<instance part="J7" gate="G$1" x="-25.4" y="83.82" rot="R180"/>
-<instance part="J6" gate="G$1" x="-25.4" y="116.84" rot="R180"/>
+<instance part="SV1" gate="1" x="66.04" y="68.58" rot="MR180">
+<attribute name="PARTNO" x="66.04" y="68.58" size="1.778" layer="96" display="off"/>
+</instance>
+<instance part="J1" gate="G$1" x="12.7" y="116.84" rot="R180">
+<attribute name="PARTNO" x="12.7" y="116.84" size="1.778" layer="96" display="off"/>
+</instance>
+<instance part="J2" gate="G$1" x="12.7" y="83.82" rot="R180">
+<attribute name="PARTNO" x="12.7" y="83.82" size="1.778" layer="96" display="off"/>
+</instance>
+<instance part="J3" gate="G$1" x="12.7" y="50.8" rot="R180">
+<attribute name="PARTNO" x="12.7" y="50.8" size="1.778" layer="96" display="off"/>
+</instance>
+<instance part="J4" gate="G$1" x="12.7" y="12.7" rot="R180">
+<attribute name="PARTNO" x="12.7" y="12.7" size="1.778" layer="96" display="off"/>
+</instance>
+<instance part="J5" gate="G$1" x="-27.94" y="5.08" rot="R180">
+<attribute name="PARTNO" x="-27.94" y="5.08" size="1.778" layer="96" display="off"/>
+</instance>
+<instance part="J8" gate="G$1" x="-25.4" y="50.8" rot="R180">
+<attribute name="PARTNO" x="-25.4" y="50.8" size="1.778" layer="96" display="off"/>
+</instance>
+<instance part="J7" gate="G$1" x="-25.4" y="83.82" rot="R180">
+<attribute name="PARTNO" x="-25.4" y="83.82" size="1.778" layer="96" display="off"/>
+</instance>
+<instance part="J6" gate="G$1" x="-25.4" y="116.84" rot="R180">
+<attribute name="PARTNO" x="-25.4" y="116.84" size="1.778" layer="96" display="off"/>
+</instance>
 <instance part="+3V1" gate="G$1" x="78.74" y="96.52"/>
 <instance part="GND1" gate="1" x="30.48" y="-15.24"/>
